File: cotti_level_shifter/cotti_level_shifter.kicad_pcb (KiCad board)
At the start: 2 copper layers, 66 x 20.3 mm, 68 parts, among them J1 Pmod GPIO 2x06 pin, J2 Pmod GPIO 2x06 socket, SW1 SW_DIP_x08, U1 74LVC1T45DW-7, U2 74LVC1T45DW-7, U3 74LVC1T45DW-7, U4 74LVC1T45DW-7, U5 74LVC1T45DW-7, U6 74LVC1T45DW-7, U7 74LVC1T45DW-7, U8 74LVC1T45DW-7

Commit message: feat: level shifter gerbers
Parts:
- removed the REF** at (142.2, 168.1)
- added REF**: cotti_logo_filled H=3mm T=0.3mm, cotti_logo:cotti_logo_filled H=3mm T=0.3mm, F.Cu at (113.5, 168.8)
- J1: footprint Pmod:Pmod_2x06_pin -> cotti_footprints:Pmod_2x06_pin
- J2: footprint Pmod:Pmod_2x06_socket -> cotti_footprints:Pmod_2x06_socket
- SW1: footprint Package_DIP:DIP-16_W7.62mm_LongPads -> cotti_footprints:SW_DS01C-254-S-08BE
- moved SW1 9.67 mm to (131.1, 166.9), turned to 0 degrees
Routing:
- net /dir4: track 29.3 -> 28.2 mm
Other:
- board text added: "A->B"
- board text added: "A<-B"
- board text added: "Rev 0.0"
- board text removed: "v0.0"
