File: cotti_level_shifter/cotti_level_shifter.kicad_sch (KiCad schematic)
At the start: 19 parts, among them J1 Pmod GPIO 2x06 pin, J2 Pmod GPIO 2x06 socket, SW1 SW_DIP_x08

Commit message: feat: level shifter gerbers
Parts:
- removed J1: Pmod GPIO 2x06 pin, Pmod:Pmod_2x06_pin, symbol Pmod:pmod_gpio_2x06_pin
- removed J2: Pmod GPIO 2x06 socket, Pmod:Pmod_2x06_socket, symbol Pmod:pmod_gpio_2x06_socket
- removed SW1: SW_DIP_x08, Package_DIP:DIP-16_W7.62mm_LongPads, symbol Switch:SW_DIP_x08
- added J1: Pmod GPIO 2x06 pin, cotti_footprints:Pmod_2x06_pin, symbol cotti_pmod:pmod_gpio_2x06_pin
- added J2: Pmod GPIO 2x06 socket, cotti_footprints:Pmod_2x06_socket, symbol cotti_pmod:pmod_gpio_2x06_socket
- added SW1: SW_DIP_x08, cotti_footprints:SW_DS01C-254-S-08BE, symbol cotti_switch:SW_DIP_x08
Connections:
- net GND: now also J1.11 (GND), J1.5 (GND), J2.11 (GND), J2.5 (GND), SW1.10, SW1.11, SW1.12, SW1.13, SW1.14, SW1.15, SW1.16, SW1.9
- net VCCA: now also J1.12 (VCC), J1.6 (VCC)
- net VCCB: now also J2.12 (VCC), J2.6 (VCC)
- net a1: now also J1.1 (IO1)
- net a2: now also J1.2 (IO2/PWM)
- net a3: now also J1.3 (IO3)
- net a4: now also J1.4 (IO4)
- net a5: now also J1.7 (IO5)
- net a6: now also J1.8 (IO6/PWM)
- net a7: now also J1.9 (IO7)
- net a8: now also J1.10 (IO8)
- net b1: now also J2.1 (IO1)
- net b2: now also J2.2 (IO2/PWM)
- net b3: now also J2.3 (IO3)
- net b4: now also J2.4 (IO4)
- net b5: now also J2.7 (IO5)
- net b6: now also J2.8 (IO6/PWM)
- net b7: now also J2.9 (IO7)
- net b8: now also J2.10 (IO8)
- net dir1: now also SW1.1
- net dir2: now also SW1.2
- net dir3: now also SW1.3
- net dir4: now also SW1.4
- net dir5: now also SW1.5
- net dir6: now also SW1.6
- net dir7: now also SW1.7
- net dir8: now also SW1.8
Other:
- note added: "Direction switch (A->B == High) A<-B == Low"
- note removed: "Direction switch (A->B == High)"
- company: (none) -> Cotti
- title: (none) -> Level Shifter Module
