File: cotti_7seg/cotti_7seg.kicad_pcb (KiCad board)
At the start: 2 copper layers, 50.8 x 20.3 mm, 40 parts, among them J1 Pmod GPIO 2x06 pin, Q1 NMOS Vth=0,7 Kp=1,5, Q10 NMOS Vth=0,7 Kp=1,5, Q11 NMOS Vth=0,7 Kp=1,5, Q12 NMOS Vth=0,7 Kp=1,5, Q13 NMOS Vth=0,7 Kp=1,5, Q14 NMOS Vth=0,7 Kp=1,5, Q15 NMOS Vth=0,7 Kp=1,5, Q16 NMOS Vth=0,7 Kp=1,5, Q2 NMOS Vth=0,7 Kp=1,5, Q3 NMOS Vth=0,7 Kp=1,5, Q4 NMOS Vth=0,7 Kp=1,5, Q5 NMOS Vth=0,7 Kp=1,5, Q6 NMOS Vth=0,7 Kp=1,5, Q7 NMOS Vth=0,7 Kp=1,5, Q8 NMOS Vth=0,7 Kp=1,5, Q9 NMOS Vth=0,7 Kp=1,5, U1 HEF4543BT_653, U2 HEF4543BT_653, U3 74LVC1G08, U4 74LVC1G08

Commit message: feat: cotti 7seg gerbers
Parts:
- removed D1, D2: 7seg Red CC, project_footprints:WL-T7DS_0.39INCH
- removed the REF** at (138.4, 67.7)
- added REF**: cotti_logo_filled H=4mm T=0.4mm, cotti_logo:cotti_logo_filled H=4mm T=0.4mm, B.Cu at (140.1, 66.7)
- added U5: 157119S12701, cotti_footprints:WL-T7DS_0.39INCH, F.Cu at (146.6, 59.9)
- added U6: SN74LVC1G08DBVR-EV, Package_TO_SOT_SMD:SOT-23-5, B.Cu at (114.3, 54.4)
- J1: footprint Pmod:Pmod_2x06_pin -> cotti_footprints:Pmod_2x06_pin
- Q1, Q10, Q11, Q12, Q13, Q14, Q15, Q16, Q2, Q3, Q4, Q5, Q6, Q7, Q8, Q9: value NMOS Vth=0,7 Kp=1,5 -> RE1C001UNTCL; footprint project_footprints:DIO_RB558WMF_ROM-L -> cotti_footprints:SOT-416
- R1, R10, R11, R12, R13, R14, R15, R16, R2, R3, R4, R5, R6, R7, R8, R9: value 62R -> 39R
- U1: value HEF4543BT_653 -> BCD_to_7seg
- U2: value HEF4543BT_653 -> 157119S12701; footprint Package_SO:SOIC-16_3.9x9.9mm_P1.27mm -> cotti_footprints:WL-T7DS_0.39INCH; moved to F.Cu
- U3: value 74LVC1G08 -> SN74LVC1G08DBVR-EV
- U4: value 74LVC1G08 -> BCD_to_7seg; footprint Package_TO_SOT_SMD:SOT-23-5 -> Package_SO:SOIC-16_3.9x9.9mm_P1.27mm
- moved U2 21.9 mm to (135.9, 59.9)
- moved Q15 9.45 mm to (120.9, 58.4), turned to -90 degrees
- moved Q13 9.37 mm to (120.9, 63.9), turned to 90 degrees
- moved U4 9.14 mm to (114.4, 63.5)
- moved Q12 7.62 mm to (128.5, 63.9), turned to 90 degrees
- moved Q8 7.55 mm to (126.0, 58.4), turned to -90 degrees
- moved Q16 7.46 mm to (126.0, 63.9), turned to 90 degrees
- moved Q7 6.04 mm to (120.9, 63.9), turned to 90 degrees
- moved Q10 5.59 mm to (126.0, 58.4), turned to -90 degrees
- moved Q5 5.08 mm to (120.9, 58.4), turned to -90 degrees
- moved Q11 2.54 mm to (128.5, 58.4), turned to -90 degrees
- moved Q6 2.54 mm to (123.4, 58.4), turned to -90 degrees
- moved Q1 0.13 mm to (123.4, 63.9), turned to 90 degrees
- moved Q14 0.13 mm to (123.4, 63.9), turned to 90 degrees
- moved Q2 0.13 mm to (126.0, 63.9), turned to 90 degrees
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Connections:
- Q1 pad 1: VCC -> /led_driver0/nmos_array0/a_in
- Q1 pad 2: /led_driver0/a -> /led_driver0/nmos_array0/a_out
- Q1 pad 3: /led_driver0/nmos_array0/a_out -> VCC
- Q10 pad 1: VCC -> /led_driver1/nmos_array0/b_in
- Q10 pad 2: /led_driver1/e -> /led_driver1/nmos_array0/b_out
- Q10 pad 3: /led_driver1/nmos_array0/e_out -> VCC
- Q11 pad 1: VCC -> /led_driver1/nmos_array0/c_in
- Q11 pad 2: /led_driver1/b -> /led_driver1/nmos_array0/c_out
- Q11 pad 3: /led_driver1/nmos_array0/b_out -> VCC
- Q12 pad 1: VCC -> /led_driver1/nmos_array0/d_in
- Q12 pad 2: /led_driver1/f -> /led_driver1/nmos_array0/d_out
- Q12 pad 3: /led_driver1/nmos_array0/f_out -> VCC
- Q13 pad 1: VCC -> /led_driver1/nmos_array0/f_in
- Q13 pad 2: /led_driver1/c -> /led_driver1/nmos_array0/f_out
- Q13 pad 3: /led_driver1/nmos_array0/c_out -> VCC
- Q14 pad 1: VCC -> /led_driver1/nmos_array0/g_in
- Q14 pad 2: /led_driver1/g -> /led_driver1/nmos_array0/g_out
- Q14 pad 3: /led_driver1/nmos_array0/g_out -> VCC
- Q15 pad 1: VCC -> /led_driver1/nmos_array0/dp_in
- Q15 pad 2: /led_driver1/d -> /led_driver1/nmos_array0/dp_out
- Q15 pad 3: /led_driver1/nmos_array0/d_out -> VCC
- Q16 pad 1: VCC -> /led_driver1/nmos_array0/e_in
- Q16 pad 2: /led_driver1/dp -> /led_driver1/nmos_array0/e_out
- Q16 pad 3: /led_driver1/nmos_array0/dp_out -> VCC
- Q2 pad 1: VCC -> /led_driver0/nmos_array0/b_in
- Q2 pad 2: /led_driver0/b -> /led_driver0/nmos_array0/b_out
- Q2 pad 3: /led_driver0/nmos_array0/b_out -> VCC
- Q3 pad 1: VCC -> /led_driver0/nmos_array0/c_in
- Q3 pad 2: /led_driver0/c -> /led_driver0/nmos_array0/c_out
- Q3 pad 3: /led_driver0/nmos_array0/c_out -> VCC
- Q4 pad 1: VCC -> /led_driver0/nmos_array0/d_in
- Q4 pad 2: /led_driver0/d -> /led_driver0/nmos_array0/d_out
- Q4 pad 3: /led_driver0/nmos_array0/d_out -> VCC
- Q5 pad 1: VCC -> /led_driver0/nmos_array0/f_in
- Q5 pad 2: /led_driver0/e -> /led_driver0/nmos_array0/f_out
- Q5 pad 3: /led_driver0/nmos_array0/e_out -> VCC
- Q6 pad 1: VCC -> /led_driver0/nmos_array0/g_in
- Q6 pad 2: /led_driver0/f -> /led_driver0/nmos_array0/g_out
- Q6 pad 3: /led_driver0/nmos_array0/f_out -> VCC
- Q7 pad 1: VCC -> /led_driver0/nmos_array0/dp_in
- Q7 pad 2: /led_driver0/g -> /led_driver0/nmos_array0/dp_out
- Q7 pad 3: /led_driver0/nmos_array0/g_out -> VCC
- Q8 pad 1: VCC -> /led_driver0/nmos_array0/e_in
- Q8 pad 2: /led_driver0/dp -> /led_driver0/nmos_array0/e_out
- Q8 pad 3: /led_driver0/nmos_array0/dp_out -> VCC
- Q9 pad 1: VCC -> /led_driver1/nmos_array0/a_in
- Q9 pad 2: /led_driver1/a -> /led_driver1/nmos_array0/a_out
- Q9 pad 3: /led_driver1/nmos_array0/a_out -> VCC
- R1 pad 2: Net-(D1-Pad10) -> Net-(U2-A)
- R2 pad 2: Net-(D1-Pad9) -> Net-(U2-B)
- R3 pad 2: Net-(D1-Pad7) -> Net-(U2-C)
- R4 pad 2: Net-(D1-Pad5) -> Net-(U2-D)
- R5 pad 2: Net-(D1-Pad4) -> Net-(U2-E)
- R6 pad 2: Net-(D1-Pad2) -> Net-(U2-F)
- R7 pad 2: Net-(D1-Pad1) -> Net-(U2-G)
- R8 pad 2: Net-(D1-Pad6) -> Net-(U2-DP)
- U1 pad 10: /led_driver0/b -> /led_driver0/nmos_array0/b_in
- U1 pad 11: /led_driver0/c -> /led_driver0/nmos_array0/c_in
- U1 pad 12: /led_driver0/d -> /led_driver0/nmos_array0/d_in
- U1 pad 13: /led_driver0/e -> /led_driver0/nmos_array0/e_in
- U1 pad 14: /led_driver0/g -> /led_driver0/nmos_array0/g_in
- U1 pad 15: /led_driver0/f -> /led_driver0/nmos_array0/f_in
- U1 pad 9: /led_driver0/a -> /led_driver0/nmos_array0/a_in
- U2 pad 1: VCC -> Net-(U2-G)
- U2 pad 10: /led_driver1/b -> Net-(U2-A)
- U2 pad 2: /d12 -> Net-(U2-F)
- U2 pad 3: /d11 -> GND
- U2 pad 4: /d13 -> Net-(U2-E)
- U2 pad 5: /d10 -> Net-(U2-D)
- U2 pad 6: GND -> Net-(U2-DP)
- U2 pad 7: GND -> Net-(U2-C)
- U2 pad 9: /led_driver1/a -> Net-(U2-B)
- U3 pad 4: /led_driver0/dp -> /led_driver0/nmos_array0/dp_in
- U4 pad 1: /d13 -> VCC
- U4 pad 3: GND -> /d11
- U4 pad 4: /led_driver1/dp -> /d13
- U4 pad 5: VCC -> /d10
Routing:
- net Net-(U2-A): track 0.00 -> 31.6 mm
- net Net-(D1-Pad10): track 31.6 -> 0.00 mm
- net Net-(U2-DP): track 0.00 -> 22.9 mm
- net Net-(D1-Pad6): track 22.9 -> 0.00 mm
- net Net-(U2-B): track 0.00 -> 22.1 mm
- net Net-(D1-Pad9): track 22.1 -> 0.00 mm
- net Net-(U2-F): track 0.00 -> 19.3 mm
- net Net-(D1-Pad2): track 19.3 -> 0.00 mm
- net /led_driver1/nmos_array0/c_in: track 0.00 -> 16.2 mm
- net /led_driver1/c: track 15.9 -> 0.00 mm
- net /led_driver1/nmos_array0/d_in: track 0.00 -> 15.7 mm
- net /led_driver1/d: track 15.5 -> 0.00 mm
- net Net-(U2-E): track 0.00 -> 15.5 mm
- net Net-(D1-Pad4): track 15.5 -> 0.00 mm
- net /led_driver0/nmos_array0/c_in: track 0.00 -> 15.1 mm
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Other:
- board text added: "Bottom row pins"
- board text added: "Rev 0.0"
- board text added: "Top row pins"
- board text removed: "v0.0"
