File: cotti_probe/cotti_probe.kicad_sch (KiCad schematic)
At the start: 45 parts, among them J1 USB_C_Receptacle_USB2.0_16P, U1 FT4232HL, U2 TLV74033PDBVR, U3 TESD5V0V4UCX6, U4 AT93C46EN, Y1 Xtal 12MHz

Commit message: feat: gerbers for cotti probe
Parts:
- removed C1: 30pF, Capacitor_SMD:C_0805_2012Metric_Pad1.18x1.45mm_HandSolder, symbol Device:C
- removed C10, C11, C12, C13, C14, C15, C16, C17, C19, C8, C9: 100nF, symbol Device:C
- removed C3: 3.3uF, symbol Device:C
- removed C4, C5: 1uF, symbol Device:C
- removed C6, C7: 4.7uF, symbol Device:C
- removed J1: USB_C_Receptacle_USB2.0_16P, symbol Connector:USB_C_Receptacle_USB2.0_16P
- removed L1, L2, L3: 2.2uH, symbol Device:L
- removed R12, R17: 5.1k, symbol Device:R_US
- removed R18, R19, R20: 10k, symbol Device:R_US
- removed R25: 2k, symbol Device:R_US
- removed TP2, TP3, TP4, TP5, TP6: TP, symbol Connector:TestPoint
- removed U2: TLV74033PDBVR, Package_TO_SOT_SMD:SOT-23-5_HandSoldering, symbol Regulator_Linear:TLV70228_SOT23-5
- removed U3: TESD5V0V4UCX6, Package_TO_SOT_SMD:SOT-23-6, symbol Power_Protection:CDSOT236-0504C
- removed U4: AT93C46EN, symbol Memory_EEPROM:93CxxB
- removed Y1: Xtal 12MHz, cotti_probe:XTAL_12MHZ, symbol Device:Crystal
- added C2: 33pF, Capacitor_SMD:C_0805_2012Metric_Pad1.18x1.45mm_HandSolder, symbol Device:C
- added Y1: XTAL 12MHz 20pF, Crystal:Crystal_SMD_HC49-SD_HandSoldering, symbol cotti_xtal:xtal_12Mhz_20pF
- C1: renamed from C2; value 30pF -> 33pF; DigiKey https://ar.mouser.com/ProductDetail/KEMET/C0805C300J4HACTU?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 -> (none); DigiKey P/N 80-C0805C300J4HACTU -> (none); Digikey (none) -> https://www.digikey.com/en/products/detail/yageo/CC0805JRNP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; Mfr. KEMET -> YAGEO; Mfr. P/N C0805C300J4HACTU -> CC0805JRNPO9BN330
- H1, H2, H3, H4: footprint (none) -> MountingHole:MountingHole_2.2mm_M2_ISO14580
- R1: footprint (none) -> Resistor_SMD:R_0805_2012Metric_Pad1.20x1.40mm_HandSolder; Digikey (none) -> https://www.digikey.com/en/products/detail/yageo/RC0805FR-1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; Mfr. (none) -> YAGEO; Mfr. P/N (none) -> RC0805FR-1012KL
- R2: renamed from R3; footprint (none) -> Resistor_SMD:R_0805_2012Metric_Pad1.20x1.40mm_HandSolder; Digikey (none) -> https://www.digikey.com/en/products/detail/yageo/RC0805FR-0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; Mfr. (none) -> YAGEO; Mfr. P/N (none) -> RC0805FR-071KL
- TP1: value TP -> TestPoint; footprint (none) -> TestPoint:TestPoint_Pad_D2.0mm
- U1: DigiKey https://www.digikey.com/en/products/detail/ftdi-future-tech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 -> (none); DigiKey P/N 768-1026-1-ND -> (none); Digikey (none) -> https://www.digikey.com/en/products/detail/ftdi-future-tech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
Connections:
- net connectors/pwren# is gone; now on net pwren#: U1.60 (~{PWREN})
- net GND: now also C2.2
- net xout: now reaches U1.3 (OSCO)
- net xout: now also C2.1, Y1.2
- net xin: now reaches C1.1, U1.2 (OSCI)
- net xin: now also Y1.1
- net VBUS renamed pwren#
- net d+ renamed D+
- net d- renamed D-
- net vphy renamed VPHY
- net vpll renamed VPLL
- no-connect marks 3 -> 1
Other:
- added sheet eeprom (eeprom.kicad_sch)
- added sheet power (power.kicad_sch)
- added sheet usb (usb.kicad_sch)
- sheet connectors ports: added none; removed eeclk, eecs, eedata, pwren#
- note added: "Crystal 12MHz"
- note removed: "Decoupling capacitors VCCIO"
- note removed: "Decoupling capacitors VCORE"
- note removed: "EEPROM"
- note removed: "LC DC filters"
- note removed: "LDO 5V -> 3.3V"
- note removed: "Test points"
- note removed: "USB and TVS protection"
- company: (none) -> Cotti
- title: (none) -> Probe Module
- moved on the sheet: C1, R1, R2, U1
