File: microprocessors/nuvoton_nuc980/boot.kicad_sch (KiCad schematic)
At the start: 22 parts, among them SW1 SW_Push_Dual, SW2 SW_DIP_x02, U6 NL17SZ17DBVT1G, Y1 XTAL 12MHz 20pF, Y2 XTAL 32.768KHz 12.5pF

Commit message: feat: ERC passing cotti-nuvoton
Parts:
- C31: footprint (none) -> Capacitor_SMD:C_0805_2012Metric_Pad1.18x1.45mm_HandSolder; Digikey (none) -> https://www.digikey.com/en/products/detail/samsung-electro-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; Mfr. (none) -> Samsung Electro-Mechanics; Mfr. P/N (none) -> CL21B474KAFNNNG
- C33, C34: footprint (none) -> Capacitor_SMD:C_0805_2012Metric_Pad1.18x1.45mm_HandSolder; Digikey (none) -> https://www.digikey.com/en/products/detail/yageo/CC0805JRNP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; Mfr. (none) -> YAGEO; Mfr. P/N (none) -> CC0805JRNPO9BN330
- C37, C38: footprint (none) -> Capacitor_SMD:C_0805_2012Metric_Pad1.18x1.45mm_HandSolder; Digikey (none) -> https://www.digikey.com/en/products/detail/yageo/CC0805JRNP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; Mfr. (none) -> YAGEO; Mfr. P/N (none) -> CC0805JRNPO9BN180
- R11, R12, R13, R14, R15, R16, R17, R20, R3, R4: footprint (none) -> Resistor_SMD:R_0805_2012Metric_Pad1.20x1.40mm_HandSolder; Digikey (none) -> https://www.digikey.com/en/products/detail/yageo/RC0805FR-1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; Mfr. (none) -> YAGEO; Mfr. P/N (none) -> RC0805FR-1310KL
- TP14, TP15: footprint (none) -> TestPoint:TestPoint_Pad_D2.0mm
