File: microprocessors/nuvoton_nuc980/nuvoton_nuc980.kicad_pcb (KiCad board)
At the start: 4 copper layers, 96.5 x 96.5 mm, 170 parts, among them J1 ADC-002-1, J11 MSD-4-A, J13 Pmod UART 2x06 socket, J14 Pmod GPIO 2x06 socket, J2 USB_C (16 + 8), J3 Pmod I2S 2x06 socket, J4 MTJ-88ARX1-LH, J5 Pmod I2C 1x06 socket, J6 Pmod GPIO 2x06 socket, J7 Pmod SPI 1x06 socket, J8 Pmod UART 1x06 socket, J9 Conn_01x10, SW1 SW_Push_Dual, SW2 SW_DIP_x02, SW3 SW_Push_Dual, T1 SM13126PEL, U1 TESD5V0V4UCX6 RFG, U10 MX30LF1G28AD-XKI, U11 TLV74312PDBVR, U12 MC74VHC1GT14DBVT1G, U13 TLV74318PDBVR, U14 NUC980DK63YC, U2 TLV74333PDBVR, U3 TPS62A01APDDCR, U4 TLV74333PDBVR, U5 MCP6541UT-E/OT, U6 NL17SZ17DBVT1G, U7 MCP6541UT-E/OT, U9 LAN8720A-CP, Y1 XTAL 12MHz 20pF, Y2 XTAL 32.768KHz 12.5pF, Y3 XTAL 25MHz 20pF

Commit message: feat: nuvoton gerber files
Parts:
- added REF**: cotti_logo_filled H=10mm T=1mm, cotti_logo:cotti_logo_filled H=10mm T=1mm, F.Cu at (135.4, 102.9)
- R22, R5, R6, R7, R8: moved to F.Cu
- moved TP16 37.7 mm to (133.1, 56.9)
- moved TP2 23.6 mm to (95.5, 71.6)
- moved TP17 17.3 mm to (106.6, 82.2)
- moved C51 12.9 mm to (142.2, 93.7), turned to -90 degrees
- moved C50 12.3 mm to (144.3, 93.7), turned to -90 degrees
- moved TP5 11.9 mm to (112.6, 69.8)
- moved R7 10.7 mm to (114.8, 58.9)
- moved R8 10.7 mm to (114.8, 56.9)
- moved TP8 10.2 mm to (93.2, 87.4)
- moved C56 10.1 mm to (150.4, 82.8), turned to 0 degrees
- moved R22 10.1 mm to (140.3, 84.3), turned to 0 degrees
- moved TP19 7.86 mm to (97.4, 133.5)
- moved R6 6.48 mm to (109.2, 58.9)
- moved TP6 6.12 mm to (116.8, 72.6)
- moved TP18 5.24 mm to (92.1, 128.7)
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Routing:
- net /GPIO4: track 113.3 -> 189.9 mm, vias 3 -> 4
- net /GPIO7: track 116.3 -> 190.7 mm
- net /GPIO2: track 116.6 -> 184.4 mm
- net /UART1_RX: track 70.4 -> 108.0 mm, vias 6 -> 4
- net /UART1_RTS: track 72.7 -> 109.0 mm, vias 6 -> 3
- net /TDO: track 56.4 -> 90.0 mm
- net /TCK: track 58.0 -> 90.6 mm
- net /TMS: track 58.0 -> 88.4 mm
- net /TDI: track 69.3 -> 96.5 mm
- net /TRST#: track 73.0 -> 99.3 mm
- net /Power/en_3.3v: track 55.8 -> 81.8 mm, vias 2 -> 6
- net +3V3: track 41.2 -> 62.6 mm, vias 14 -> 62
- net /rst#: track 176.4 -> 197.7 mm, vias 10 -> 6
- net /UART1_CTS: track 81.1 -> 101.9 mm, vias 6 -> 3
- net /I2C2_SCL: track 66.4 -> 86.3 mm, vias 6 -> 4
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- added copper zone on B.Cu, net +1V8
- added copper zone on F.Cu, net +1V8
- added copper zone on B.Cu, net +2V2
Other:
- board text added: "0"
- board text added: "1"
- board text added: "B0"
- board text added: "B1"
- board text added: "Boot Mode"
- board text added: "GPIOs"
- board text added: "I2S"
- board text added: "Nuvoton NUC980DK63YC"
- board text added: "RESET"
- board text added: "Rev 0.0"
- board text added: "USER BTN"
- board text added: "USER LED"
